File: sonar-usart-3led/sonar-usart-3led.kicad/sonar-usart-3led.sch (KiCad schematic (older format))
At the start: 10 parts, among them IC1 ATTINY2313-P

Commit message: Update kicad files for the sonar-usart-3led schematic. not complete, external oscillator needs to be updated. pin conflict on tiny and sonar ground?
Parts:
- added Y?: Crystal, symbol Crystal
- Q1: renamed from Q?; symbol PN2222A -> PN2222A-RESCUE-sonar-usart-3led
- gave numbers to parts that had none: 4
Connections:
- net labels removed: Earth
- wire segments 36 -> 30
- no-connect marks 14 -> 17
Changed lines of the file:
@@
 L GND #PWR03
 U 1 1 5633A646
-P 4050 3500
-F 0 "#PWR03" H 4050 3250 50  0001 C CNN
-F 1 "GND" H 4050 3350 50  0000 C CNN
-F 2 "" H 4050 3500 60  0000 C CNN
-F 3 "" H 4050 3500 60  0000 C CNN
-	1    4050 3500
+P 3600 3400
+F 0 "#PWR03" H 3600 3150 50  0001 C CNN
+F 1 "GND" H 3600 3250 50  0000 C CNN
+F 2 "" H 3600 3400 60  0000 C CNN
+F 3 "" H 3600 3400 60  0000 C CNN
+	1    3600 3400
 	1    0    0    -1
 $EndComp
 $Comp
-L LV-MaxSonar-EZ1 U?
+L LV-MaxSonar-EZ1 U1
 U 1 1 56462BB2
 P 5300 4550
-F 0 "U?" H 5300 4550 60  0000 C CNN
+F 0 "U1" H 5300 4550 60  0000 C CNN
 F 1 "LV-MaxSonar-EZ1" H 5300 4550 60  0000 C CNN
 F 2 "" H 5300 4550 60  0000 C CNN
@@
 NoConn ~ 5200 4350
 Connection ~ 6450 2250
-Wire Wire Line
-	3600 3400 5100 3400
-Wire Wire Line
-	3800 3400 3800 3500
-Wire Wire Line
-	3800 3500 4050 3500
 Wire Wire Line
 	5700 2050 5850 2050
@@
 	3900 1300 3900 1050
 Wire Wire Line
-	5100 3400 5100 3850
-Wire Wire Line
 	5100 3850 5200 3850
-Connection ~ 3800 3400
 Wire Wire Line
 	1850 1300 1850 3950
@@
 	1850 3950 5200 3950
 Connection ~ 3600 1300
-Wire Wire Line
-	5200 4450 4700 4450
-Wire Wire Line
-	4700 4450 4700 3400
-Connection ~ 4700 3400
 $Comp
-L PN2222A Q?
+L PN2222A-RESCUE-sonar-usart-3led Q1
 U 1 1 56C25F47
 P 3650 4800
-F 0 "Q?" H 3850 4875 50  0000 L CNN
+F 0 "Q1" H 3850 4875 50  0000 L CNN
 F 1 "PN2222A" H 3850 4800 50  0000 L CNN
 F 2 "TO-92" H 3850 4725 50  0000 L CIN
@@
 $EndComp
 $Comp
-L R R?
+L R R6
 U 1 1 56C26029
 P 3750 4250
-F 0 "R?" V 3830 4250 50  0000 C CNN
+F 0 "R6" V 3830 4250 50  0000 C CNN
 F 1 "R 10 kOhm" V 3650 4250 50  0000 C CNN
 F 2 "" V 3680 4250 30  0000 C CNN
@@
 $EndComp
 $Comp
-L R R?
+L R R4
 U 1 1 56C26271
 P 3000 4800
-F 0 "R?" V 3080 4800 50  0000 C CNN
+F 0 "R4" V 3080 4800 50  0000 C CNN
 F 1 "R 10 kOhm" V 2900 4800 50  0000 C CNN
 F 2 "" V 2930 4800 30  0000 C CNN
@@
 $EndComp
 $Comp
-L R R?
+L R R5
 U 1 1 56C262D8
 P 3300 5150
-F 0 "R?" V 3380 5150 50  0000 C CNN
+F 0 "R5" V 3380 5150 50  0000 C CNN
 F 1 "R 10 kOhm" V 3200 5150 50  0000 C CNN
 F 2 "" V 3230 5150 30  0000 C CNN
@@
 $EndComp
 Wire Wire Line
-	3450 4800 3150 4800
+	3150 4800 3450 4800
 Wire Wire Line
 	3300 5000 3300 4800
 Connection ~ 3300 4800
-$Comp
-L Earth #PWR?
-U 1 1 56C2650C
-P 3500 5400
-F 0 "#PWR?" H 3500 5150 50  0001 C CNN
-F 1 "Earth" H 3500 5250 50  0001 C CNN
-F 2 "" H 3500 5400 60  0000 C CNN
-F 3 "" H 3500 5400 60  0000 C CNN
-	1    3500 5400
-	1    0    0    -1
-$EndComp
 Wire Wire Line
 	3750 5400 3750 5000
@@
 Connection ~ 3750 3950
 Wire Wire Line
-	3750 4600 3750 4400
+	3750 4400 3750 4600
 Wire Wire Line
 	5200 4050 2850 4050
@@
 	4900 2500 4750 2500
 Connection ~ 3750 4500
+NoConn ~ 5200 4150
+NoConn ~ 4750 2000
+$Comp
+L GND #PWR04
+U 1 1 57773EA1
+P 3500 5400
+F 0 "#PWR04" H 3500 5150 50  0001 C CNN
+F 1 "GND" H 3500 5250 50  0000 C CNN
+F 2 "" H 3500 5400 60  0000 C CNN
+F 3 "" H 3500 5400 60  0000 C CNN
+	1    3500 5400
+	1    0    0    -1
+$EndComp
+NoConn ~ 5200 4450
+$Comp
+L GND #PWR05
+U 1 1 57774512
+P 5100 3850
+F 0 "#PWR05" H 5100 3600 50  0001 C CNN
+F 1 "GND" H 5100 3700 50  0000 C CNN
+F 2 "" H 5100 3850 50  0000 C CNN
+F 3 "" H 5100 3850 50  0000 C CNN
+	1    5100 3850
+	0    1    1    0
+$EndComp
+$Comp
+L Crystal Y?
+U 1 1 57774800
+P 2150 2000
+F 0 "Y?" H 2150 2150 50  0000 C CNN
+F 1 "Crystal" H 2150 1850 50  0000 C CNN
+F 2 "" H 2150 2000 50  0000 C CNN
+F 3 "" H 2150 2000 50  0000 C CNN
+	1    2150 2000
+	0    1    1    0
+$EndComp
 $EndSCHEMATC
